File: pcb/cl0ck_control/cl0ck_control.kicad_pcb (KiCad board)
At the start: 2 copper layers, 307 x 27 mm, 16 parts, among them CON1 AVR-ISP-6, IC1 ATMEGA328P-A, IC2 DS3234, P1 CONN_01X03, P2 CONN_01X02, P3 GPS, SW1 SW_RESET, SW2 SW_B1, SW3 SW_B2

Commit message: Revision to control pcb.
Parts:
- added REF**: MountingHole_3.2mm_M3_Pad, Mounting_Holes:MountingHole_3.2mm_M3_Pad, F.Cu at (62.2, 130.8)
- added REF**: MountingHole_3.2mm_M3_Pad, Mounting_Holes:MountingHole_3.2mm_M3_Pad, F.Cu at (62.2, 145.8)
- added REF**: MountingHole_3.2mm_M3_Pad, Mounting_Holes:MountingHole_3.2mm_M3_Pad, F.Cu at (357.2, 145.8)
- added REF**: MountingHole_3.2mm_M3_Pad, Mounting_Holes:MountingHole_3.2mm_M3_Pad, F.Cu at (357.2, 130.8)
- C2: moved to B.Cu
- CON1: value AVR-ISP-6 -> AVR-ISP
- PH2: value BUTTON_CONN -> BUTTONS
- POWER1: value BARREL_JACK -> 5V
- SW2: value SW_B1 -> B1
- SW3: value SW_B2 -> B2
- moved SW3 178.8 mm to (201.2, 137.8), turned to 180 degrees
- moved P2 177.9 mm to (276.2, 132.8)
- moved P1 177.1 mm to (276.2, 137.8)
- moved RESET 173.2 mm to (251.2, 144.8)
- moved PH2 171.9 mm to (180.2, 142.8)
- moved R1 170.6 mm to (243.0, 146.2), turned to 90 degrees
- moved POWER1 170.4 mm to (89.2, 138.8)
- moved CON1 170.3 mm to (248.2, 132.8), turned to 90 degrees
- moved P3 168.5 mm to (137.2, 142.8)
- moved IC1 167.7 mm to (227.2, 137.8)
- moved PH1 166.5 mm to (110.2, 142.8)
- moved C1 166.4 mm to (218.2, 137.4), turned to 90 degrees
- moved SW2 165.3 mm to (164.2, 137.8), turned to 180 degrees
- moved IC2 159.9 mm to (310.2, 137.8)
- moved BATT 159.3 mm to (337.2, 137.8)
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- renumbered BATT1 to BATT, SW1 to RESET
Routing:
- net VCC: track 74.4 -> 291.3 mm, vias 3 -> 4
- net uCU_RXD: track 0.00 -> 124.7 mm, vias 0 -> 2
- net uCU_TXD: track 0.00 -> 121.4 mm, vias 0 -> 2
- net MOSI: track 37.0 -> 137.3 mm, vias 4 -> 5
- net SS: track 0.00 -> 97.5 mm, vias 0 -> 2
- net BUTT_1: track 0.00 -> 91.6 mm
- net MISO: track 26.6 -> 117.0 mm, vias 3 -> 2
- net BUTT_2: track 0.00 -> 84.9 mm
- net SCK: track 49.3 -> 118.5 mm, vias 4 -> 3
- net +BATT: track 0.00 -> 37.9 mm
- net GND: track 0.00 -> 32.9 mm, vias 0 -> 4
- net LOAD_SEGS: track 40.4 -> 63.6 mm, vias 3 -> 2
- net 'RESET: track 43.9 -> 56.9 mm, vias 2 -> 4
- added copper zone on B.Cu, net GND
- added copper zone on F.Cu, net GND
Other:
- board text added: "DISPLAY"
- board text added: "GND"

Commit message: Revised control schematic and PCB files.  Finalised and ordered first trial run.
Parts:
- removed BATT: 3V, Battery_Holders:Keystone_3000_1x12mm-CoinCell
- removed RESET: SW_RESET, Buttons_Switches_SMD:SW_SPST_PTS645
- added BATT1: 3V, Battery_Holders:Keystone_3000_1x12mm-CoinCell, B.Cu at (337.2, 137.8)
- added SW1: SW_RESET, Buttons_Switches_SMD:SW_SPST_PTS645, B.Cu at (251.2, 144.8)
- CON1: value AVR-ISP -> AVR-ISP-6
- P1: footprint Pin_Headers:Pin_Header_Angled_1x03 -> Pin_Headers:Pin_Header_Straight_1x03
- P2: footprint Pin_Headers:Pin_Header_Angled_1x02 -> Pin_Headers:Pin_Header_Straight_1x02
- P3: footprint Pin_Headers:Pin_Header_Angled_1x05 -> Pin_Headers:Pin_Header_Straight_1x05
- PH2: value BUTTONS -> BUTTON_CONN
- POWER1: value 5V -> BARREL_JACK
- SW2: value B1 -> SW_B1
- SW3: value B2 -> SW_B2
- moved PH1 17.0 mm to (93.2, 142.8)
- moved P3 13.6 mm to (150.8, 142.8), turned to 180 degrees
- moved POWER1 10.4 mm to (78.8, 138.8)
- moved C2 2.80 mm to (301.0, 138.8)
- moved C1 1.20 mm to (219.4, 137.4)
Connections:
- IC1 pad 1: Net-(IC1-Pad1) -> (no net)
- IC1 pad 10: Net-(IC1-Pad10) -> (no net)
- IC1 pad 11: Net-(IC1-Pad11) -> (no net)
- IC1 pad 12: Net-(IC1-Pad12) -> (no net)
- IC1 pad 19: Net-(IC1-Pad19) -> (no net)
- IC1 pad 2: Net-(IC1-Pad2) -> (no net)
- IC1 pad 20: Net-(IC1-Pad20) -> (no net)
- IC1 pad 22: Net-(IC1-Pad22) -> (no net)
- IC1 pad 25: Net-(IC1-Pad25) -> (no net)
- IC1 pad 26: Net-(IC1-Pad26) -> (no net)
- IC1 pad 27: Net-(IC1-Pad27) -> (no net)
- IC1 pad 28: Net-(IC1-Pad28) -> (no net)
- IC1 pad 32: Net-(IC1-Pad32) -> (no net)
- IC1 pad 7: Net-(IC1-Pad7) -> (no net)
- IC1 pad 8: Net-(IC1-Pad8) -> (no net)
- IC1 pad 9: Net-(IC1-Pad9) -> (no net)
- IC2 pad 3: Net-(IC2-Pad3) -> (no net)
- IC2 pad 5: Net-(IC2-Pad5) -> (no net)
- IC2 pad 6: Net-(IC2-Pad6) -> (no net)
- P3 pad 1: Net-(P3-Pad1) -> (no net)
- PH1 pad 2: Net-(PH1-Pad2) -> (no net)
- PH1 pad 6: Net-(PH1-Pad6) -> (no net)
- POWER1 pad 3: Net-(POWER1-Pad3) -> (no net)
Routing:
- net uCU_RXD: track 124.7 -> 191.4 mm
- net uCU_TXD: track 121.4 -> 180.8 mm
- net VCC: track 291.3 -> 284.2 mm
Other:
- board text added: "gps_cl0ck"
- board text added: "jadon_clews 2018"
