File: pcb/cl0ck_control/cl0ck_control.sch (KiCad schematic (older format))
At the start: 14 parts, among them CON1 AVR-ISP-6, IC1 ATMEGA328P-A, IC2 DS3234, P1 CONN_01X03, P2 CONN_01X02, SW1 SW_RESET, SW2 SW_B1, SW3 SW_B2

Commit message: Working on control pcb.
Parts:
- added P3: GPS, Pin_Headers:Pin_Header_Angled_1x05, symbol CONN_01X05
- added POWER1: BARREL_JACK, Connectors:BARREL_JACK, symbol BARREL_JACK
- P1: footprint (none) -> Pin_Headers:Pin_Header_Angled_1x03
- P2: footprint (none) -> Pin_Headers:Pin_Header_Angled_1x02
- PH1: footprint Pin_Headers:Pin_Header_Straight_1x06 -> Pin_Headers:Pin_Header_Angled_1x06
- PH2: footprint Pin_Headers:Pin_Header_Straight_1x03 -> Pin_Headers:Pin_Header_Angled_1x03
Connections:
- net GND: now also P3.4 (P4), POWER1.2
- net VCC: now also P3.5 (P5), POWER1.1
- net uCU_RXD: now also P3.3 (P3)
- net uCU_TXD: now also P3.2 (P2)
- no-connect marks 21 -> 23
Changed lines of the file:
@@
 F 0 "PH1" H 5200 6150 50  0000 C CNN
 F 1 "FTDI" V 5300 5800 50  0000 C CNN
-F 2 "Pin_Headers:Pin_Header_Straight_1x06" H 5200 5800 50  0001 C CNN
+F 2 "Pin_Headers:Pin_Header_Angled_1x06" H 5200 5800 50  0001 C CNN
 F 3 "" H 5200 5800 50  0000 C CNN
 	1    5200 5800
@@
 F 0 "PH2" H 7300 1900 50  0000 C CNN
 F 1 "BUTTON_CONN" V 7400 1700 50  0000 C CNN
-F 2 "Pin_Headers:Pin_Header_Straight_1x03" H 7300 1700 50  0001 C CNN
+F 2 "Pin_Headers:Pin_Header_Angled_1x03" H 7300 1700 50  0001 C CNN
 F 3 "" H 7300 1700 50  0000 C CNN
 	1    7300 1700
@@
 F 0 "P1" H 6400 3800 50  0000 C CNN
 F 1 "CONN_01X03" V 6500 3600 50  0000 C CNN
-F 2 "" H 6400 3600 50  0000 C CNN
+F 2 "Pin_Headers:Pin_Header_Angled_1x03" H 6400 3600 50  0001 C CNN
 F 3 "" H 6400 3600 50  0000 C CNN
 	1    6400 3600
@@
 F 0 "P2" H 6400 4350 50  0000 C CNN
 F 1 "CONN_01X02" V 6500 4200 50  0000 C CNN
-F 2 "" H 6400 4200 50  0000 C CNN
+F 2 "Pin_Headers:Pin_Header_Angled_1x02" H 6400 4200 50  0001 C CNN
 F 3 "" H 6400 4200 50  0000 C CNN
 	1    6400 4200
@@
 Wire Wire Line
 	6700 4250 6700 4300
+$Comp
+L CONN_01X05 P3
+U 1 1 5B279B47
+P 2750 5850
+F 0 "P3" H 2750 6150 50  0000 C CNN
+F 1 "GPS" V 2850 5850 50  0000 C CNN
+F 2 "Pin_Headers:Pin_Header_Angled_1x05" H 2750 5850 50  0001 C CNN
+F 3 "" H 2750 5850 50  0000 C CNN
+	1    2750 5850
+	-1   0    0    1
+$EndComp
+$Comp
+L BARREL_JACK POWER1
+U 1 1 5B279BCE
+P 2000 5700
+F 0 "POWER1" H 2000 5950 50  0000 C CNN
+F 1 "BARREL_JACK" H 2000 5500 50  0000 C CNN
+F 2 "Connectors:BARREL_JACK" H 2000 5700 50  0001 C CNN
+F 3 "" H 2000 5700 50  0000 C CNN
+	1    2000 5700
+	1    0    0    -1
+$EndComp
+Text GLabel 3050 6000 2    60   Input ~ 0
+uCU_TXD
+Text GLabel 3050 5850 2    60   Input ~ 0
+uCU_RXD
+$Comp
+L VCC #PWR025
+U 1 1 5B279E3B
+P 3650 5600
+F 0 "#PWR025" H 3650 5450 50  0001 C CNN
+F 1 "VCC" H 3650 5750 50  0000 C CNN
+F 2 "" H 3650 5600 50  0000 C CNN
+F 3 "" H 3650 5600 50  0000 C CNN
+	1    3650 5600
+	1    0    0    -1
+$EndComp
+$Comp
+L GND #PWR026
+U 1 1 5B279EB6
+P 3650 5800
+F 0 "#PWR026" H 3650 5550 50  0001 C CNN
+F 1 "GND" H 3650 5650 50  0000 C CNN
+F 2 "" H 3650 5800 50  0000 C CNN
+F 3 "" H 3650 5800 50  0000 C CNN
+	1    3650 5800
+	1    0    0    -1
+$EndComp
+NoConn ~ 2950 6050
+Wire Wire Line
+	3050 6000 3000 6000
+Wire Wire Line
+	3000 6000 3000 5950
+Wire Wire Line
+	3000 5950 2950 5950
+Wire Wire Line
+	2950 5850 3050 5850
+Wire Wire Line
+	2950 5750 3650 5750
+Wire Wire Line
+	3650 5750 3650 5800
+Wire Wire Line
+	3650 5600 3650 5650
+Wire Wire Line
+	3650 5650 2950 5650
+$Comp
+L VCC #PWR027
+U 1 1 5B27A23F
+P 2450 5500
+F 0 "#PWR027" H 2450 5350 50  0001 C CNN
+F 1 "VCC" H 2450 5650 50  0000 C CNN
+F 2 "" H 2450 5500 50  0000 C CNN
+F 3 "" H 2450 5500 50  0000 C CNN
+	1    2450 5500
+	1    0    0    -1
+$EndComp
+$Comp
+L GND #PWR028
+U 1 1 5B27A27A
+P 2450 5900
+F 0 "#PWR028" H 2450 5650 50  0001 C CNN
+F 1 "GND" H 2450 5750 50  0000 C CNN
+F 2 "" H 2450 5900 50  0000 C CNN
+F 3 "" H 2450 5900 50  0000 C CNN
+	1    2450 5900
+	1    0    0    -1
+$EndComp
+NoConn ~ 2300 5700
+Wire Wire Line
+	2450 5500 2450 5600
+Wire Wire Line
+	2450 5600 2300 5600
+Wire Wire Line
+	2300 5800 2450 5800
+Wire Wire Line
+	2450 5800 2450 5900
 $EndSCHEMATC

Commit message: Revised control schematic and PCB files.  Finalised and ordered first trial run.
Parts:
- P1: footprint Pin_Headers:Pin_Header_Angled_1x03 -> Pin_Headers:Pin_Header_Straight_1x03
- P2: footprint Pin_Headers:Pin_Header_Angled_1x02 -> Pin_Headers:Pin_Header_Straight_1x02
- P3: footprint Pin_Headers:Pin_Header_Angled_1x05 -> Pin_Headers:Pin_Header_Straight_1x05
Changed lines of the file:
@@
 F 0 "P1" H 6400 3800 50  0000 C CNN
 F 1 "CONN_01X03" V 6500 3600 50  0000 C CNN
-F 2 "Pin_Headers:Pin_Header_Angled_1x03" H 6400 3600 50  0001 C CNN
+F 2 "Pin_Headers:Pin_Header_Straight_1x03" H 6400 3600 50  0001 C CNN
 F 3 "" H 6400 3600 50  0000 C CNN
 	1    6400 3600
@@
 F 0 "P2" H 6400 4350 50  0000 C CNN
 F 1 "CONN_01X02" V 6500 4200 50  0000 C CNN
-F 2 "Pin_Headers:Pin_Header_Angled_1x02" H 6400 4200 50  0001 C CNN
+F 2 "Pin_Headers:Pin_Header_Straight_1x02" H 6400 4200 50  0001 C CNN
 F 3 "" H 6400 4200 50  0000 C CNN
 	1    6400 4200
@@
 F 0 "P3" H 2750 6150 50  0000 C CNN
 F 1 "GPS" V 2850 5850 50  0000 C CNN
-F 2 "Pin_Headers:Pin_Header_Angled_1x05" H 2750 5850 50  0001 C CNN
+F 2 "Pin_Headers:Pin_Header_Straight_1x05" H 2750 5850 50  0001 C CNN
 F 3 "" H 2750 5850 50  0000 C CNN
 	1    2750 5850
